File: Pressure_Board.sch (KiCad schematic (older format))
At the start: 10 parts, among them J1 Conn_01x01, J2 Conn_01x02, K1 RELAY-1XCHANGE_SPDT_RevE_Date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, T1 TRANSISTOR-NPN-BIPOLAR_EN6061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, U1 HSC_Sensor

Commit message: Add files via upload
Parts:
- removed J1: Conn_01x01, symbol Conn_01x01
- added J1: Conn_01x02, symbol Conn_01x02
- added J3: Barrel_Jack, symbol Barrel_Jack
- added U3: LF90_TO252, TO_SOT_Packages_THT:TO-252-2, symbol LF90_TO252
- gave numbers to parts that had none: 2
Connections:
- net +12V: now also J3.1, U3.1 (VI)
- net GND: now also J1.2 (Pin_2), J3.2, J3.3, U3.2 (GND)
- net D3: now reaches SHIELD1.3
- net D3: now also U2.13 (DB6)
- net D4: now reaches SHIELD1.4
- net D4: now also U2.12 (DP5)
- net D5: now reaches SHIELD1.5
- net D5: now also U2.11 (DP4)
- net D6: now reaches SHIELD1.6
- net D6: now also U2.14 (DB7)
- net D7: now reaches SHIELD1.7
- net D7: now also U2.6 (EN)
- net D8: now reaches SHIELD1.8
- net D8: now also U2.4 (RS)
- net V_IN: now reaches SHIELD1.V_IN
- net V_IN: now also U3.3 (VO)
- net at K1.11: now also J1.1 (Pin_1)
Other:
- moved on the sheet: D1, J2, K1, R1, SHIELD1, T1, U1, U2, U4
